File: kicad/tanekonsat2022_auto.kicad_sch (KiCad schematic)
At the start: 84 parts

Commit message: schematic circuit diagram (almost) done!
Parts:
- removed C? (x2): 10u, Capacitor_SMD:C_0805_2012Metric, symbol Device:C
- removed C?: 0.01u, symbol Device:C_Small
- removed C?: 0.1u, symbol Device:C_Small
- removed C? (x2): 1u, symbol Device:C_Small
- removed IC?: NJM2884U1-33-TE1, SOT-89-5-1, symbol SamacSys_Parts:NJM2884U1-33-TE1
- removed IC?: CGGBPD.25.A, SamacSys_Parts:CGGBPD25A, symbol SamacSys_Parts:CGGBPD.25.A
- removed IC?: PCA9306D, SamacSys_Parts:SOIC127P600X175-8N, symbol SamacSys_Parts:PCA9306D
- removed IC?: NJM12877F33-TE1, SamacSys_Parts:SOT95P280X120-5N, symbol SamacSys_Parts:NJM12877F33-TE1
- removed R? (x2): 2.2k, symbol Device:R_Small
- removed R? (x2): 3.3k, symbol Device:R_Small
- removed R?: 200k, symbol Device:R_Small
- removed U?: ICM-20948_SL, tanekonsat:ICM-20948_SL, symbol tanekonsat:ICM-20948_SL
- removed U?: AZ1117-3.3, SamacSys_Parts:SOT230P700X180-4N, symbol Regulator_Linear:AZ1117-3.3
- added C16, C24, C25, C27, C28, C29, C9: (no value), symbol Device:C_Small
- added C18, C19, C20, C21: (no value), symbol Device:C
- added FL1: (no value), symbol SamacSys_Parts:SAFEA1G58KA0F00R15
- added IC5: (no value), symbol SamacSys_Parts:CGGBPD.25.A
- added IC6: (no value), symbol SamacSys_Parts:MAX2641EUT+T
- added J4: (no value), symbol Connector:Conn_01x02_Male
- added J5, J6: (no value), symbol Connector:Conn_01x06_Female
- added J7: (no value), symbol Connector:Conn_01x04_Female
- added L1, L2: (no value), symbol Device:L
- added Q7: (no value), symbol Device:Q_NMOS_DGS
- added R22, R23: (no value), symbol Device:R
- C1, C10, C11, C12, C13, C15, C3, C6, C8: renamed from C?; value 0.1u -> (none); footprint Capacitor_SMD:C_0402_1005Metric -> (none); LCSC (none) -> C1525
- C14: renamed from C?; value 0.1u -> (none); LCSC (none) -> C1525
- C17: renamed from C?; value 0.1u -> (none); LCSC (none) -> C52923
- C2, C5: renamed from C?; value 27p -> (none); footprint Capacitor_SMD:C_0402_1005Metric -> (none); LCSC (none) -> C1557
- C22: renamed from C?; value 0.1u -> (none); LCSC (none) -> C15195
- C23: renamed from C?; value 1u -> (none); LCSC (none) -> C52923
- C26: renamed from C?; value 56p -> (none); LCSC (none) -> C39148
- C4, C7: renamed from C?; value 1u -> (none); footprint Capacitor_SMD:C_0402_1005Metric -> (none); LCSC (none) -> C52923
- D1, D2: renamed from D?; value SS2040FL_R1_00001 -> (none); footprint SODFL3618X110N -> (none)
- D3: renamed from D?; value LED -> (none)
- IC1: renamed from IC?; value W25Q128JVSIQ -> (none); footprint SamacSys_Parts:SOIC127P790X216-8N -> (none); LCSC (none) -> C97521
- IC2: renamed from IC?; value ADP3338AKCZ-3.3-RL -> (none); footprint SOT230P700X180-4N -> (none)
- IC3: renamed from IC?; value NJM12888F18 -> (none); footprint SamacSys_Parts:SOT95P280X130-5N -> (none)
- IC4: renamed from IC?; value TESEO-LIV3F -> (none); footprint SamacSys_Parts:SON110P970X1010X230-18N -> (none)
- IC7, IC8: renamed from IC?; value TB67H450FNG,EL -> (none); footprint SOIC127P600X175-9N -> (none)
- J1: renamed from J?; value Conn_01x02_Male -> (none); footprint Connector_JST:JST_PH_S3B-PH-K_1x03_P2.00mm_Horizontal -> (none)
- J2: renamed from J?; value USB_B_Micro -> (none); footprint SamacSys_Parts:ZX62R-B-5P_30_ -> (none)
- J3: renamed from J?; value Conn_01x02_Male -> (none)
- M1, M2: renamed from M?; value Motor_DC -> (none)
- Q1, Q2: renamed from Q?; value Q_NMOS_DGS -> (none); footprint SamacSys_Parts:SOT95P237X112-3N -> (none)
- Q3, Q4, Q5, Q6: renamed from Q?; value BSS138 -> (none); footprint SOT95P240X120-3N -> (none)
- R1, R10, R11, R12, R13, R14, R15, R16, R17, R3, R9: renamed from R?; value 10k -> (none); LCSC (none) -> C25744
- R18, R19, R20, R21: renamed from R?; value R -> (none)
- R2, R4: renamed from R?; value 1k -> (none); footprint Capacitor_SMD:C_0402_1005Metric -> (none); LCSC (none) -> C11702
- R5, R6: renamed from R?; value 27 -> (none); footprint Capacitor_SMD:C_0402_1005Metric -> (none); LCSC (none) -> C25771
- R7: renamed from R?; value 660 -> (none); LCSC (none) -> C11702
- R8: renamed from R?; value 1k -> (none); LCSC (none) -> C11702
- S1, S2: renamed from S?; value SKRPACE010 -> (none); footprint SamacSys_Parts:SMT_4.2X3.2_ -> (none)
- SW1: renamed from SW?; value SW_DIP_x01 -> (none); footprint SamacSys_Parts:SSAJ120100 -> (none)
- U1: renamed from U?; value RP2040 -> (none); footprint RP2040:RP2040-QFN-56 -> (none); LCSC (none) -> C2040
- U2: renamed from U?; value CR2032 -> (none); footprint tanekonsat:CR2032 -> (none)
- U3: renamed from U?; value VL53L5X_SL -> (none)
- U4: renamed from U?; value ICM-20948_SL -> (none); footprint tanekonsat:ICM-20948_SL -> (none)
- Y1: renamed from Y?; value FA-238V_12.0000MB-K3 -> (none); footprint SamacSys_Parts:FA238V120000MBK3 -> (none)
Connections:
- net GPIO13 is gone; now on net GPIO13_MO_A_2: U1.16 (GPIO13)
- net GPIO14 is gone; now on net GPIO14_MO_B_1: U1.17 (GPIO14)
- net GPIO15 is gone; now on net GPIO15_MO_B_2: U1.18 (GPIO15)
- net GPIO2 is gone; now on net GPIO2_ToF_RST: U1.4 (GPIO2)
- net GPIO3 is gone; now on net GPIO3_Nichrome: U1.5 (GPIO3)
- net GPIO8 is gone; now on net GPIO8_ToF_SDA: U1.11 (GPIO8)
- net GPIO9 is gone; now on net GPIO9_ToF_SCL: U1.12 (GPIO9)
- net M_CS is gone; now on net GPIO17_M_CS: Q6.3, R13.2
- net M_SCLK is gone; now on net GPIO18_M_SCK: Q3.3, R10.2
- net M_SDI is gone; now on net GPIO19_M_SDI_RX: Q4.3, R11.2
- net M_SDO is gone; now on net GPIO16_M_SDO_TX: Q5.3, R12.2
- net +3V3: now also C16.1, C20.1, C21.1, C29.1, C29.2, C9.1, IC6.6 (VCC), J5.3 (Pin_3), J6.3 (Pin_3), J7.2 (Pin_2)
- net +7V4: now also C18.1, J4.1 (Pin_1)
- net GND: now also C16.2, C18.2, C19.2, C20.2, C21.2, C9.2, J5.6 (Pin_6), J6.6 (Pin_6), Q7.2 (S), R23.2
- net GND2: now also C24.2, FL1.2 (GND_1), FL1.3 (GND_2), FL1.5 (GND_3), IC6.2 (GND_1), IC6.3 (GND_2), IC6.5 (GND_3), J7.1 (Pin_1), L2.2
- net GPIO4_GNSS_TX: now also J7.3 (Pin_3)
- net GPIO5_GNSS_RX: now also J7.4 (Pin_4)
- net V_REG: now also C19.1
- net GPIO14_MO_B_1: now reaches IC8.2 (IN2)
- net GPIO14_MO_B_1: now also J6.1 (Pin_1)
- net GPIO15_MO_B_2: now reaches IC8.3 (IN1)
- net GPIO15_MO_B_2: now also J6.2 (Pin_2)
- net GPIO13_MO_A_2: now reaches IC7.2 (IN2)
- net GPIO13_MO_A_2: now also IC7.3 (IN1), J5.1 (Pin_1), J5.2 (Pin_2)
- net GPIO9_ToF_SCL: now reaches U3.2 (SCL)
- net GPIO2_ToF_RST: now reaches U3.3 (RST)
- net GPIO8_ToF_SDA: now reaches U3.4 (SDA)
- net at IC4.11 (RF_IN): now also C27.2
- net GPIO3_Nichrome: now reaches R8.1
- net GPIO12 renamed GPIO12_MO_A_1
- net GPIO16 renamed GPIO16_M_SDO_TX
- net GPIO17 renamed GPIO17_M_CS
- net GPIO18 renamed GPIO18_M_SCK
- net GPIO19 renamed GPIO19_M_SDI_RX
- net GPIO20 renamed GPIO20_MOE_A_1
- net GPIO21 renamed GPIO21_MOE_A_2
- net GPIO22 renamed GPIO22_MOE_B_1
- net GPIO22_MOE_B_1: now also J6.4 (Pin_4)
- net GPIO23 renamed GPIO23_MOE_B_2
- net GPIO23_MOE_B_2: now also J6.5 (Pin_5)
- net GPIO24 renamed GPIO24_Nichrome
- net GPIO24_Nichrome: now also R22.1
- new net: J4.2 (Pin_2), Q7.3 (D)
- new net: C24.1, C25.1, IC5.1
- new net: C25.2, L1.1
- new net: C28.2, FL1.1 (IN), L2.1
- new net: C27.1, FL1.4 (OUT)
- new net: IC6.1 (RFIN), L1.2
- new net: Q7.1 (G), R22.2, R23.1
- new net: C28.1, IC6.4 (RFOUT)
- new net GPIO20_MOE_A_2: J5.5 (Pin_5)
- new net GPIO21_MOE_A_1: J5.4 (Pin_4)
Other:
- note added: "GPIO16: SPI0 RX"
- note added: "GPIO19: SPI0 TX"
- note added: "Power(Conn)"
- note added: "Run SW"
- note added: "USB"
- note removed: "I2C（SDA, SCL）をRP2040と接続する I2CよりSPIの方がよいか…"
- note removed: "Run SW（出来れば載せる）"
- note removed: "レギュレーターを一つにしてダイオードで切り替えにする"
- note removed: "秋月で在庫切れ"
- moved on the sheet: C10, C11, C12, C13, C15, C26, C8, IC4, IC7, IC8, J3, M1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

Commit message: done! AW of GNSS board
Parts:
- removed C26: (no value), symbol Device:C_Small
- added J8: (no value), symbol Connector:Conn_01x02_Female
- C19, C20, C21: LCSC C15008 -> (none)
- C2, C5: LCSC C1557 -> C32949
Connections:
- net GPIO20_MOE_A_2 is gone; now on net GPIO21_MOE_A_2: J5.5 (Pin_5)
- net GPIO21_MOE_A_1 is gone; now on net GPIO20_MOE_A_1: J5.4 (Pin_4)
- net +3V3: no longer C29.1, C29.2, IC6.6 (VCC)
- net GND2: now also C29.2
- net GPIO12_MO_A_1: now also IC7.3 (IN1)
- net GPIO13_MO_A_2: no longer IC7.3 (IN1), J5.1 (Pin_1), J5.2 (Pin_2)
- net GPIO14_MO_B_1: now also IC8.3 (IN1); no longer IC8.2 (IN2), J6.1 (Pin_1)
- net GPIO15_MO_B_2: now also IC8.2 (IN2); no longer IC8.3 (IN1), J6.2 (Pin_2)
- net M2_MINUS: now reaches IC8.6 (OUT1), M2.2 (-)
- net M2_MINUS: now also J6.2 (Pin_2)
- net M2_PLUS: now reaches IC8.8 (OUT2), M2.1 (+)
- net M2_PLUS: now also J6.1 (Pin_1)
- net M1_MINUS: now reaches IC7.6 (OUT1), M1.2 (-)
- net M1_MINUS: now also J5.2 (Pin_2)
- net M1_PLUS: now reaches IC7.8 (OUT2), M1.1 (+)
- net M1_PLUS: now also J5.1 (Pin_1)
- net VCC_RF: now reaches IC4.14 (VCC_RF)
- net VCC_RF: now also C29.1, IC6.6 (VCC)
- net at IC4.16 (SDA): now also J8.2 (Pin_2)
- net at IC4.17 (SCL): now also J8.1 (Pin_1)
Other:
- note added: "Pin8(VCC)とPin14(VCC_RF)は内部的に接続されている"
- moved on the sheet: IC7, IC8, J5, J6, M1, M2, R18, R19, R20, R21
