File: kicad/tanekonsat2022_auto.kicad_sch (KiCad schematic)
At the start: 94 parts

Commit message: done AW of main board
Parts:
- removed C31, C32: (no value), symbol Device:C
- removed J5, J6: (no value), symbol Connector:Conn_01x06_Female
- removed R24, R25, R26, R27: (no value), symbol Device:R
- removed U4: (no value), symbol Isolator:LTV-824
- removed Y1: (no value), symbol SamacSys_Parts:FA-238V_12.0000MB-K3
- added C17, C22, C23: 100u, Capacitor_SMD:C_1206_3216Metric, symbol Device:C
- added J5, J6: Conn_01x04_Male, tanekonsat:PinHeader_1x04_P2.00mm_Vertical, symbol Connector:Conn_01x04_Male
- added R12: 100, Capacitor_SMD:C_0603_1608Metric, symbol Device:R
- added R13, R15: 1k, Capacitor_SMD:C_0603_1608Metric, symbol Device:R
- added R14: 3k, Capacitor_SMD:C_0603_1608Metric, symbol Device:R
- added U5: LT6106, Package_TO_SOT_SMD:SOT-23-5, symbol Amplifier_Current:LT6106
- added U6: Opamp_Dual, Package_SO:SSOP-8_5.25x5.24mm_P1.27mm, symbol Device:Opamp_Dual
- added Y1: SIT2001BI-S2-33E-12.000000D, Package_TO_SOT_SMD:SOT-23-5, symbol SamacSys_Parts:SIT2001BI-S2-33E-12.000000D
- AC1: value (none) -> BNO085; footprint (none) -> SamacSys_Parts:BNO085
- C1, C10, C11, C12, C13, C14, C15, C3, C34, C37, C6, C8: value (none) -> 100n; footprint (none) -> Capacitor_SMD:C_0603_1608Metric
- C16, C4, C7, C9: value (none) -> 1u; footprint (none) -> Capacitor_SMD:C_0603_1608Metric
- C18, C19, C20, C21, C26, C30, C33: value (none) -> 100u; footprint (none) -> Capacitor_SMD:C_1206_3216Metric
- C2: value (none) -> 10p; footprint (none) -> Capacitor_SMD:C_0603_1608Metric
- C24: value (none) -> 1p; footprint (none) -> Capacitor_SMD:C_0603_1608Metric
- C25, C28: value (none) -> 100p; footprint (none) -> Capacitor_SMD:C_0603_1608Metric
- C27: value (none) -> 120p; footprint (none) -> Capacitor_SMD:C_0603_1608Metric
- C29: value (none) -> 470p; footprint (none) -> Capacitor_SMD:C_0603_1608Metric
- C35, C36: value (none) -> 22p; footprint (none) -> Capacitor_SMD:C_0603_1608Metric
- C5: value (none) -> 100u; footprint (none) -> Capacitor_SMD:C_1206_3216Metric; LCSC C32949 -> (none)
- D1: value (none) -> 1N4148W; footprint (none) -> Diode_SMD:D_SOD-123
- D3: value (none) -> LED; footprint (none) -> Capacitor_SMD:C_0603_1608Metric
- FL1: value (none) -> SAFEA1G58KA0F00R15; footprint (none) -> SamacSys_Parts:SAFEA1G58KA0F00R15
- IC1: value (none) -> W25Q128JVSIQ; footprint (none) -> SamacSys_Parts:SOIC127P790X216-8N
- IC2: value (none) -> ADP3338AKCZ-3.3-RL; footprint (none) -> SamacSys_Parts:SOT230P700X180-4N
- IC4: value (none) -> TESEO-LIV3F; footprint (none) -> SamacSys_Parts:SON110P970X1010X230-18N
- IC5: value (none) -> CGGBPD.25.A; footprint (none) -> SamacSys_Parts:CGGBPD25A
- IC6: value (none) -> MAX2641EUT+T; footprint (none) -> SamacSys_Parts:SOT95P280X145-6N
- IC7, IC8: value (none) -> TB67H450FNG,EL; footprint (none) -> SamacSys_Parts:SOIC127P600X175-9N
- J1: value (none) -> Conn_01x02_Male; footprint (none) -> Connector_JST:JST_PH_S3B-PH-K_1x03_P2.00mm_Horizontal
- J10, J9: value (none) -> Conn_01x05_Female; footprint (none) -> tanekonsat:PinHeader_1x05_P2.00mm_Vertical
- J11: value (none) -> Conn_01x02_Female; footprint (none) -> tanekonsat:PinHeader_1x02_P2.00mm_Vertical
- J12: value (none) -> Conn_01x02_Female
- J2: value (none) -> USB_B_Micro; footprint (none) -> SamacSys_Parts:101181940001LFBKN
- J3, J4: value (none) -> Conn_01x02_Male; footprint (none) -> tanekonsat:PinHeader_1x02_P2.00mm_Vertical
- J7: value (none) -> Conn_01x04_Female; footprint (none) -> tanekonsat:PinHeader_1x04_P2.00mm_Vertical
- J8: value (none) -> Conn_01x02_Female; footprint (none) -> Connector_PinHeader_2.00mm:PinHeader_1x02_P2.00mm_Vertical
- L1: value (none) -> 5.6n; footprint (none) -> Inductor_SMD:L_0603_1608Metric_Pad1.05x0.95mm_HandSolder
- L2: value (none) -> 6.8n; footprint (none) -> Inductor_SMD:L_0603_1608Metric_Pad1.05x0.95mm_HandSolder
- M1, M2: value (none) -> Motor_DC; footprint (none) -> tanekonsat:PinHeader_1x02_P2.00mm_Vertical
- Q1, Q2, Q7: value (none) -> Q_NMOS_DGS; footprint (none) -> SamacSys_Parts:SOT95P237X112-3N
- R1, R11, R23, R9: value (none) -> 10k; footprint (none) -> Capacitor_SMD:C_0603_1608Metric
- R10: value (none) -> 0.01; footprint (none) -> Resistor_SMD:R_1206_3216Metric
- R18, R19, R20, R21: value (none) -> R; footprint (none) -> Resistor_SMD:R_0603_1608Metric_Pad0.98x0.95mm_HandSolder
- R2, R22, R7, R8: value (none) -> 1k; footprint (none) -> Capacitor_SMD:C_0603_1608Metric
- R3: value (none) -> DNF; footprint (none) -> Resistor_SMD:R_0603_1608Metric_Pad0.98x0.95mm_HandSolder
- R4: value (none) -> 10k; footprint (none) -> Capacitor_SMD:C_0603_1608Metric; LCSC C11702 -> C25744
- R5, R6: value (none) -> 27; footprint (none) -> Capacitor_SMD:C_0603_1608Metric
- S1, S2: value (none) -> SKRPACE010; footprint (none) -> SamacSys_Parts:SMT_4.2X3.2_
- SW1: value (none) -> SW_DIP_x01; footprint (none) -> SamacSys_Parts:SSAJ120100
- U1: value (none) -> RP2040; footprint (none) -> RP2040:RP2040-QFN-56
- U2: value (none) -> CR1025; footprint (none) -> tanekonsat:CR1025_Holder
- U3: value (none) -> VL53L5X_SL
- Y2: value (none) -> FC-135_32.768KHz_7pF_+_-20ppm; footprint (none) -> SamacSys_Parts:FC-135
Connections:
- net GND2 is gone; now on net GND: C24.2, C29.2, FL1.2 (GND_1), FL1.3 (GND_2), FL1.5 (GND_3), IC4.1 (GND), IC4.10 (GND_RF_1), IC4.12 (GND_RF_2), IC6.2 (GND_1), IC6.3 (GND_2), IC6.5 (GND_3), J7.1 (Pin_1), J9.1 (Pin_1), L2.2, U2.1 (minus)
- net +3V3: now also AC1.28 (VDDIO), AC1.3 (VDD), C33.1, C37.1, R10.2, C17.1, C23.1, J5.4 (Pin_4), J6.4 (Pin_4), U5.4 (+), U6.8 (V+), Y1.4 (VDD); no longer C16.1, C9.1, IC2.2 (OUT_1), IC2.4 (OUT_2)
- net +7V4: now also C5.1, C22.1, R14.2; no longer C33.1
- net GND: now also AC1.10 (CLKSEL0), AC1.2 (GND_1), AC1.25 (GND_2), C2.2, IC7.1 (GND), IC8.1 (GND), R18.1, R19.1, R20.1, R21.1, C17.2, C22.2, C23.2, J5.1 (Pin_1), J6.1 (Pin_1), R13.2, R15.1, U5.2 (V-), U6.4 (V-), Y1.1 (GND); no longer C2.1, R10.1
- net GPIO20_MOE_A_1: now also J6.3 (Pin_3)
- net GPIO23_MOE_B_2: now also J5.2 (Pin_2)
- net XIN: now also C2.1, Y1.5 (OUT); no longer C2.2
- net XOUT: no longer R4.1
- net at R4.2: now also Q1.1 (G); no longer C5.1
- net GPIO10_MO_A_1: now reaches IC7.3 (IN1)
- net GPIO10_MO_A_1: now also U1.13 (GPIO10)
- net GPIO11_MO_A_2: now reaches IC7.2 (IN2)
- net GPIO11_MO_A_2: now also U1.14 (GPIO11)
- net GPIO19_MO_B_2: now reaches IC8.2 (IN2)
- net GPIO19_MO_B_2: now also U1.30 (GPIO19)
- net GPIO18_MO_B_1: now reaches IC8.3 (IN1)
- net GPIO18_MO_B_1: now also U1.29 (GPIO18)
- net at R1.1, SW1.C1: now also R4.1; no longer Q1.1 (G)
- net GPIO7_ToF_SCL: now reaches U3.2 (SCL)
- net GPIO7_ToF_SCL: now also J10.1 (Pin_1), U1.9 (GPIO7)
- net GPIO3_ToF_RST: now reaches U3.3 (RST)
- net GPIO3_ToF_RST: now also J10.2 (Pin_2), U1.5 (GPIO3)
- net GPIO6_ToF_SDA: now reaches U3.4 (SDA)
- net GPIO6_ToF_SDA: now also J10.3 (Pin_3), U1.8 (GPIO6)
- removed net GND3: IC7.1 (GND), IC8.1 (GND), R10.2, R18.1, R19.1, R20.1, R21.1
- net GPIO10_I2C_EXT_SDA renamed GPIO8_I2C_EXT_SDA
- net GPIO8_I2C_EXT_SDA: now also U1.11 (GPIO8); no longer U1.13 (GPIO10)
- net GPIO11_I2C_EXT_SCL renamed GPIO9_I2C_EXT_SCL
- net GPIO9_I2C_EXT_SCL: now also U1.12 (GPIO9); no longer U1.14 (GPIO11)
- net GPIO12_MO_A_1 renamed GPIO12_IMU_MISO
- net GPIO12_IMU_MISO: now also AC1.20 (H_SDA/H_MISO/TX), J12.1 (Pin_1)
- net GPIO13_MO_A_2 renamed GPIO13_IMU_CS
- net GPIO13_IMU_CS: now also AC1.18 (H_CSN)
- net GPIO14_MO_B_1 renamed GPIO14_IMU_SCK
- net GPIO14_IMU_SCK: now also AC1.19 (H_SCL/SCK/RX), J12.2 (Pin_2)
- net GPIO15_MO_B_2 renamed GPIO15_IMU_MOSI
- net GPIO15_IMU_MOSI: now also AC1.17 (SA0/H_MOSI)
- removed net GPIO16_IMU_MISO: AC1.20 (H_SDA/H_MISO/TX), J12.1 (Pin_1), U1.27 (GPIO16)
- net GPIO17_IMU_CS renamed GPIO17_IMU_RST
- net GPIO17_IMU_RST: now also AC1.11 (NRST); no longer AC1.18 (H_CSN)
- removed net GPIO18_IMU_SCK: AC1.19 (H_SCL/SCK/RX), J12.2 (Pin_2), U1.29 (GPIO18)
- removed net GPIO19_IMU_MOSI: AC1.17 (SA0/H_MOSI), U1.30 (GPIO19)
- net GPIO21_MOE_A_2 renamed GPIO21_MOE_B_1
- net GPIO21_MOE_B_1: now also J5.3 (Pin_3)
- net GPIO22_MOE_B_1 renamed GPIO22_MOE_A_2
- net GPIO22_MOE_A_2: now also J6.2 (Pin_2)
- net GPIO24_NichromeB: no longer names the net of U1.36 (GPIO24)
- net GPIO24_NichromeB: no longer R22.1
- net GPIO25_NichromeA: no longer names the net of U1.37 (GPIO25)
- net GPIO25_NichromeA: no longer R8.1
- net GPIO26_ADC0 renamed GPIO26_ADC_I_monitor
- net GPIO26_ADC_I_monitor: now also U6.1, U6.2 (-)
- net GPIO27_ADC1 renamed GPIO27_ADC_V_monitor
- net GPIO27_ADC_V_monitor: now also U6.6 (-), U6.7
- net GPIO28_ADC2 renamed GPIO28_NichromeA
- net GPIO28_NichromeA: now also R8.1
- net GPIO29_ADC3 renamed GPIO29_NichromeB
- net GPIO29_NichromeB: now also R22.1
- net GPIO2_ToF_RST renamed GPIO2_LED
- net GPIO2_LED: now also R7.1; no longer J10.2 (Pin_2)
- removed net GPIO3_LED: R7.1, U1.5 (GPIO3)
- net GPIO6_IMU_INT renamed GPIO16_IMU_INT
- net GPIO16_IMU_INT: now also U1.27 (GPIO16); no longer U1.8 (GPIO6)
- removed net GPIO7_IMU_RST: AC1.11 (NRST), U1.9 (GPIO7)
- removed net GPIO8_ToF_SDA: J10.3 (Pin_3), U1.11 (GPIO8)
- removed net GPIO9_ToF_SCL: J10.1 (Pin_1), U1.12 (GPIO9)
- new net: R14.1, R15.2, U6.5 (+)
- new net: R13.1, U5.1, U6.3 (+)
- new net: R12.2, U5.3 (-)
- new net 3V3_REG_OUT: C16.1, C9.1, IC2.2 (OUT_1), IC2.4 (OUT_2), R10.1, R12.1, U5.5 (V+)
Other:
- note added: "GPIO12: SPI1 RX"
- note added: "GPIO15: SPI1 TX"
- note added: "Pin8(VCC)とPin14(VCC_RF)は内部で接続されている"
- note added: "Power(monitor)"
- note added: "Vadc = Vbat / 3"
- note added: "connect after draw"
- note removed: "GPIO16: SPI0 RX"
- note removed: "GPIO19: SPI0 TX"
- note removed: "Pin8(VCC)とPin14(VCC_RF)は内部的に接続されている"
- moved on the sheet: C20, C24, C25, C27, C28, C29, C33, D3, FL1, IC4, IC5, IC6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

Commit message: update conn
Parts:
- removed J2: USB_B_Micro, SamacSys_Parts:101181940001LFBKN, symbol RP2040_minimal-rescue:USB_B_Micro-Connector
- added R16, R17: (no value), symbol Device:R
- added U4: (no value), symbol tanekonsat:USB_type_C
- AC1: value BNO085 -> (none); footprint SamacSys_Parts:BNO085 -> (none)
- C1, C10, C11, C12, C13, C14, C15, C3, C34, C37, C6, C8: value 100n -> (none); footprint Capacitor_SMD:C_0603_1608Metric -> (none)
- C16, C4, C7, C9: value 1u -> (none); footprint Capacitor_SMD:C_0603_1608Metric -> (none)
- C17, C18, C19, C20, C21, C22, C23, C26, C30, C33, C5: value 100u -> (none); footprint Capacitor_SMD:C_1206_3216Metric -> (none)
- C2: value 10p -> (none); footprint Capacitor_SMD:C_0603_1608Metric -> (none)
- C24: value 1p -> (none); footprint Capacitor_SMD:C_0603_1608Metric -> (none)
- C25, C28: value 100p -> (none); footprint Capacitor_SMD:C_0603_1608Metric -> (none)
- C27: value 120p -> (none); footprint Capacitor_SMD:C_0603_1608Metric -> (none)
- C29: value 470p -> (none); footprint Capacitor_SMD:C_0603_1608Metric -> (none)
- C35, C36: value 22p -> (none); footprint Capacitor_SMD:C_0603_1608Metric -> (none)
- D1: value 1N4148W -> (none); footprint Diode_SMD:D_SOD-123 -> (none)
- D3: value LED -> (none); footprint Capacitor_SMD:C_0603_1608Metric -> (none)
- FL1: value SAFEA1G58KA0F00R15 -> (none); footprint SamacSys_Parts:SAFEA1G58KA0F00R15 -> (none)
- IC1: value W25Q128JVSIQ -> (none); footprint SamacSys_Parts:SOIC127P790X216-8N -> (none)
- IC2: value ADP3338AKCZ-3.3-RL -> (none); footprint SamacSys_Parts:SOT230P700X180-4N -> (none)
- IC4: value TESEO-LIV3F -> (none); footprint SamacSys_Parts:SON110P970X1010X230-18N -> (none)
- IC5: value CGGBPD.25.A -> (none); footprint SamacSys_Parts:CGGBPD25A -> (none)
- IC6: value MAX2641EUT+T -> (none); footprint SamacSys_Parts:SOT95P280X145-6N -> (none)
- IC7, IC8: value TB67H450FNG,EL -> (none); footprint SamacSys_Parts:SOIC127P600X175-9N -> (none)
- J1: value Conn_01x02_Male -> (none); footprint Connector_JST:JST_PH_S3B-PH-K_1x03_P2.00mm_Horizontal -> (none)
- J10, J9: value Conn_01x05_Female -> (none); footprint tanekonsat:PinHeader_1x05_P2.00mm_Vertical -> (none)
- J11: value Conn_01x02_Female -> (none); footprint tanekonsat:PinHeader_1x02_P2.00mm_Vertical -> (none)
- J12: value Conn_01x02_Female -> (none)
- J3, J4: value Conn_01x02_Male -> (none); footprint tanekonsat:PinHeader_1x02_P2.00mm_Vertical -> (none)
- J5, J6: value Conn_01x04_Male -> (none); footprint tanekonsat:PinHeader_1x04_P2.00mm_Vertical -> (none)
- J7: value Conn_01x04_Female -> (none); footprint tanekonsat:PinHeader_1x04_P2.00mm_Vertical -> (none)
- J8: value Conn_01x02_Female -> (none); footprint Connector_PinHeader_2.00mm:PinHeader_1x02_P2.00mm_Vertical -> (none)
- L1: value 5.6n -> (none); footprint Inductor_SMD:L_0603_1608Metric_Pad1.05x0.95mm_HandSolder -> (none)
- L2: value 6.8n -> (none); footprint Inductor_SMD:L_0603_1608Metric_Pad1.05x0.95mm_HandSolder -> (none)
- M1, M2: value Motor_DC -> (none); footprint tanekonsat:PinHeader_1x02_P2.00mm_Vertical -> (none)
- Q1, Q2, Q7: value Q_NMOS_DGS -> (none); footprint SamacSys_Parts:SOT95P237X112-3N -> (none)
- R1, R11, R23, R4, R9: value 10k -> (none); footprint Capacitor_SMD:C_0603_1608Metric -> (none)
- R10: value 0.01 -> (none); footprint Resistor_SMD:R_1206_3216Metric -> (none)
- R12: value 100 -> (none); footprint Capacitor_SMD:C_0603_1608Metric -> (none)
- R13, R15, R2, R22, R7, R8: value 1k -> (none); footprint Capacitor_SMD:C_0603_1608Metric -> (none)
- R14: value 3k -> (none); footprint Capacitor_SMD:C_0603_1608Metric -> (none)
- R18, R19, R20, R21: value R -> (none); footprint Resistor_SMD:R_0603_1608Metric_Pad0.98x0.95mm_HandSolder -> (none)
- R3: value DNF -> (none); footprint Resistor_SMD:R_0603_1608Metric_Pad0.98x0.95mm_HandSolder -> (none)
- R5, R6: value 27 -> (none); footprint Capacitor_SMD:C_0603_1608Metric -> (none)
- S1, S2: value SKRPACE010 -> (none); footprint SamacSys_Parts:SMT_4.2X3.2_ -> (none)
- SW1: value SW_DIP_x01 -> (none); footprint SamacSys_Parts:SSAJ120100 -> (none)
- U1: value RP2040 -> (none); footprint RP2040:RP2040-QFN-56 -> (none)
- U2: value CR1025 -> (none); footprint tanekonsat:CR1025_Holder -> (none)
- U3: value VL53L5X_SL -> (none)
- U5: value LT6106 -> (none); footprint Package_TO_SOT_SMD:SOT-23-5 -> (none)
- U6: value Opamp_Dual -> (none); footprint Package_SO:SSOP-8_5.25x5.24mm_P1.27mm -> (none)
- Y1: value SIT2001BI-S2-33E-12.000000D -> (none); footprint Package_TO_SOT_SMD:SOT-23-5 -> (none)
- Y2: value FC-135_32.768KHz_7pF_+_-20ppm -> (none); footprint SamacSys_Parts:FC-135 -> (none)
Connections:
- net GND: now also R16.2, R17.2, U4.1 (A1-B12_GND), U4.12 (A12-B1_GND), U4.SHIELD
- net USB_D+: now also U4.6 (A6_DP1), U4.8 (B6_DP2)
- net USB_D-: now also U4.5 (B7_DN2), U4.7 (A7_DN1)
- net VBUS: now also U4.11 (A9-B4_VBUS), U4.2 (A4-B9_VBUS)
- new net: R16.1, U4.10 (B5_CC2)
- new net: R17.1, U4.4 (A5_CC1)
- no-connect marks 1 -> 0
