File: kicad/tanekonsat2022_auto_0905.kicad_sch (KiCad schematic)
At the start: 94 parts

Commit message: update 9-axis sensor
Parts:
- removed C34, C35, C36, C37: (no value), symbol Device:C_Small
- removed D1: (no value), symbol Diode:1N4148W
- removed J11, J12: (no value), symbol Connector:Conn_01x02_Female
- removed R10, R11, R24, R25, R26, R27: (no value), symbol Device:R
- removed U4: (no value), symbol Isolator:LTV-824
- removed Y2: (no value), symbol SamacSys_Parts:FC-135_32.768KHz_7pF_+_-20ppm
- added C17, C23: 1u, Capacitor_SMD:C_0402_1005Metric, symbol Device:C_Small
- added C22: 0.01u, Capacitor_SMD:C_0402_1005Metric, symbol Device:C_Small
- added D1, D2: SS2040FL_R1_00001, SamacSys_Parts:SODFL3618X110N, symbol SamacSys_Parts:SS2040FL_R1_00001
- added IC3: NJM12888F18, SamacSys_Parts:SOT95P280X130-5N, symbol SamacSys_Parts:NJM12888F05
- added Q3, Q4, Q5, Q6: BSS138, SamacSys_Parts:SOT95P240X120-3N, symbol SamacSys_Parts:BSS138
- added R10, R11, R12, R13, R14, R15, R16, R17: 10k, Resistor_SMD:R_0402_1005Metric, symbol Device:R_Small
- added U4: ICM-20948_SL, tanekonsat:ICM-20948_SL, symbol tanekonsat:ICM-20948_SL
- C1, C10, C11, C12, C13, C14, C15, C3, C6, C8: value (none) -> 100n; footprint (none) -> Capacitor_SMD:C_0402_1005Metric
- C16, C4, C7, C9: value (none) -> 1u; footprint (none) -> Capacitor_SMD:C_0402_1005Metric
- C18, C19, C20, C21, C26, C30, C31, C32, C33: value (none) -> 100u; footprint (none) -> Capacitor_SMD:C_1206_3216Metric
- C2, C5: value (none) -> 10p; footprint (none) -> Capacitor_SMD:C_0402_1005Metric
- C24: value (none) -> 1p; footprint (none) -> Capacitor_SMD:C_0402_1005Metric
- C25, C28: value (none) -> 100p; footprint (none) -> Capacitor_SMD:C_0402_1005Metric
- C27: value (none) -> 120p; footprint (none) -> Capacitor_SMD:C_0402_1005Metric
- C29: value (none) -> 470p; footprint (none) -> Capacitor_SMD:C_0402_1005Metric
- D3: value (none) -> LED; footprint (none) -> Capacitor_SMD:C_0603_1608Metric_Pad1.08x0.95mm_HandSolder
- FL1: value (none) -> SAFEA1G58KA0F00R15; footprint (none) -> SamacSys_Parts:SAFEA1G58KA0F00R15
- IC1: value (none) -> W25Q128JVSIQ; footprint (none) -> SamacSys_Parts:SOIC127P790X216-8N
- IC2: value (none) -> ADP3338AKCZ-3.3-RL; footprint (none) -> SamacSys_Parts:SOT230P700X180-4N
- IC4: value (none) -> TESEO-LIV3F; footprint (none) -> SamacSys_Parts:SON110P970X1010X230-18N
- IC5: value (none) -> CGGBPD.25.A; footprint (none) -> SamacSys_Parts:CGGBPD25A
- IC6: value (none) -> MAX2641EUT+T; footprint (none) -> SamacSys_Parts:SOT95P280X145-6N
- IC7, IC8: value (none) -> TB67H450FNG,EL; footprint (none) -> SamacSys_Parts:SOIC127P600X175-9N
- J1: value (none) -> Conn_01x02_Male; footprint (none) -> Connector_JST:JST_PH_S3B-PH-K_1x03_P2.00mm_Horizontal
- J10, J9: value (none) -> Conn_01x05_Female; footprint (none) -> tanekonsat:PinHeader_1x05_P2.00mm_Vertical
- J2: value (none) -> USB_B_Micro; footprint (none) -> SamacSys_Parts:101181940001LFBKN
- J3, J4: value (none) -> Conn_01x02_Male; footprint (none) -> tanekonsat:PinHeader_1x02_P2.00mm_Vertical
- J5, J6: value (none) -> Conn_01x06_Female; footprint (none) -> tanekonsat:PinHeader_1x06_P2.00mm_Vertical
- J7: value (none) -> Conn_01x04_Female; footprint (none) -> tanekonsat:PinHeader_1x04_P2.00mm_Vertical
- J8: value (none) -> Conn_01x02_Female; footprint (none) -> Connector_PinHeader_2.00mm:PinHeader_1x02_P2.00mm_Vertical
- L1: value (none) -> 5.6n; footprint (none) -> Inductor_SMD:L_0603_1608Metric_Pad1.05x0.95mm_HandSolder
- L2: value (none) -> 6.8n; footprint (none) -> Inductor_SMD:L_0603_1608Metric_Pad1.05x0.95mm_HandSolder
- M1, M2: value (none) -> Motor_DC
- Q1, Q2, Q7: value (none) -> Q_NMOS_DGS; footprint (none) -> SamacSys_Parts:SOT95P237X112-3N
- R1, R23, R9: value (none) -> 10k; footprint (none) -> Resistor_SMD:R_0402_1005Metric
- R18, R19, R20, R21: value (none) -> R; footprint (none) -> Resistor_SMD:R_0603_1608Metric_Pad0.98x0.95mm_HandSolder
- R2, R22, R4, R8: value (none) -> 1k; footprint (none) -> Resistor_SMD:R_0402_1005Metric
- R3: value (none) -> DNF; footprint (none) -> Resistor_SMD:R_0603_1608Metric_Pad0.98x0.95mm_HandSolder
- R5, R6: value (none) -> 27; footprint (none) -> Resistor_SMD:R_0402_1005Metric
- R7: value (none) -> 660; footprint (none) -> Resistor_SMD:R_0402_1005Metric
- S1, S2: value (none) -> SKRPACE010; footprint (none) -> SamacSys_Parts:SMT_4.2X3.2_
- SW1: value (none) -> SW_DIP_x01; footprint (none) -> SamacSys_Parts:SSAJ120100
- U1: value (none) -> RP2040; footprint (none) -> RP2040:RP2040-QFN-56
- U2: value (none) -> CR1025; footprint (none) -> tanekonsat:CR1025_Holder
- U3: value (none) -> VL53L5X_SL
- Y1: value (none) -> FA-238V_12.0000MB-K3; footprint (none) -> SamacSys_Parts:FA238V120000MBK3
- renumbered AC1 to AC?
Connections:
- net +3V3: now also C17.1, IC3.1 (VIN), IC3.3 (CONTROL), R10.1, R11.1, R12.1, R13.1
- net +7V4: now also D1.2; no longer C19.1, IC2.3 (IN)
- net GND: now also C17.2, C22.1, C23.2, IC3.2 (GND), U4.9 (INT)
- net GPIO12_MO_A_1: now also IC7.3 (IN1)
- net GPIO13_MO_A_2: now also IC7.2 (IN2)
- net GPIO14_MO_B_1: now also IC8.3 (IN1)
- net GPIO15_MO_B_2: now also IC8.2 (IN2)
- net VBUS: now also D2.2
- net at AC?.28 (VDDIO): no longer AC?.3 (VDD)
- net GPIO10_I2C_EXT_SDA renamed GPIO10
- net GPIO11_I2C_EXT_SCL renamed GPIO11
- net GPIO16_IMU_MISO: no longer names the net of AC?.20 (H_SDA/H_MISO/TX)
- net GPIO16_IMU_MISO: no longer U1.27 (GPIO16)
- net GPIO17_IMU_CS: no longer names the net of AC?.18 (H_CSN)
- net GPIO17_IMU_CS: no longer U1.28 (GPIO17)
- net GPIO18_IMU_SCK: no longer names the net of AC?.19 (H_SCL/SCK/RX)
- net GPIO18_IMU_SCK: no longer U1.29 (GPIO18)
- net GPIO19_IMU_MOSI: no longer names the net of AC?.17 (SA0/H_MOSI)
- net GPIO19_IMU_MOSI: no longer U1.30 (GPIO19)
- net GPIO6_IMU_INT: no longer names the net of AC?.14 (H_INTN)
- net GPIO6_IMU_INT: no longer U1.8 (GPIO6)
- net GPIO7_IMU_RST: no longer names the net of AC?.11 (NRST)
- net GPIO7_IMU_RST: no longer U1.9 (GPIO7)
- new net: C22.2, IC3.4 (CS)
- new net +1V8: C23.1, IC3.5 (VOUT), Q3.1, Q4.1, Q5.1, Q6.1, R14.1, R15.1, R16.1, R17.1, U4.1 (VDD), U4.2 (VDDIO)
- new net GPIO16_M_SDO_TX: Q5.3, R12.2, U1.27 (GPIO16)
- new net GPIO17_M_CS: Q6.3, R13.2, U1.28 (GPIO17)
- new net GPIO18_M_SCK: Q3.3, R10.2, U1.29 (GPIO18)
- new net GPIO19_M_SDI_RX: Q4.3, R11.2, U1.30 (GPIO19)
- new net GPIO6: U1.8 (GPIO6)
- new net GPIO7: U1.9 (GPIO7)
- new net IMU_CS: Q6.2, R17.2, U4.6 (CS)
- new net IMU_SCLK: Q3.2, R14.2, U4.3 (SCL/SCLK)
- new net IMU_SDI: Q4.2, R15.2, U4.4 (SDA/SDI)
- new net IMU_SDO: Q5.2, R16.2, U4.5 (AD0/SDO)
- new net V_REG: C19.1, D1.1, D2.1, IC2.3 (IN)
- now unconnected: AC?.4 (BOOTN), AC?.5 (PS1), AC?.6 (PS0/WAKE)
Other:
- note added: "LV(Low Voltage)側に1V8， HV(High Voltage)側に3V3 GNDは直結でよい"
- note added: "NJM12888F18はVinが6V5までなので，効率悪いけど3V3から取っている．"
- note added: "SPIレベル変換回路"
- note added: "USB"
- note removed: "EXTEND I2C"
- moved on the sheet: AC?, C24, C25, C27, C28, C29, D3, FL1, IC4, IC5, IC6, IC7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
