File: kicad2/prometheus-em/prometheus-em.kicad_sch (KiCad schematic)
At the start: 78 parts

Commit message: update pcb
Changed lines of the file:
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@@
       (effects (font (size 1.27 1.27)) hide)
     )
-    (property "Value" "" (id 1) (at 308.61 224.79 0))
+    (property "Value" "GND" (id 1) (at 308.61 224.79 0))
     (property "Footprint" "" (id 2) (at 308.61 220.98 0)
       (effects (font (size 1.27 1.27)) hide)
@@
       (effects (font (size 1.27 1.27)) hide)
     )
-    (property "Value" "" (id 1) (at 180.34 45.72 0))
+    (property "Value" "+1V8" (id 1) (at 180.34 45.72 0))
     (property "Footprint" "" (id 2) (at 180.34 49.53 0)
       (effects (font (size 1.27 1.27)) hide)
@@
       (effects (font (size 1.27 1.27)) hide)
     )
-    (property "Value" "" (id 1) (at 309.88 63.5 0))
+    (property "Value" "GND" (id 1) (at 309.88 63.5 0))
     (property "Footprint" "" (id 2) (at 309.88 59.69 0)
       (effects (font (size 1.27 1.27)) hide)
@@
       (effects (font (size 1.27 1.27)) hide)
     )
-    (property "Value" "" (id 1) (at 35.56 252.73 0))
+    (property "Value" "GND" (id 1) (at 35.56 252.73 0))
     (property "Footprint" "" (id 2) (at 35.56 248.92 0)
       (effects (font (size 1.27 1.27)) hide)
@@
       (effects (font (size 1.27 1.27)) hide)
     )
-    (property "Value" "" (id 1) (at 279.4 44.45 0))
+    (property "Value" "GNDA" (id 1) (at 279.4 44.45 0))
     (property "Footprint" "" (id 2) (at 279.4 40.64 0)
       (effects (font (size 1.27 1.27)) hide)
@@
       (effects (font (size 1.27 1.27)) hide)
     )
-    (property "Value" "" (id 1) (at 289.56 173.99 0))
+    (property "Value" "GND" (id 1) (at 289.56 173.99 0))
     (property "Footprint" "" (id 2) (at 289.56 170.18 0)
       (effects (font (size 1.27 1.27)) hide)

Commit message: complete prometheus-em pcb
Parts:
- removed U2: (no value), symbol tanekonsat:ICM-20948
- added C22, C23: (no value), symbol Device:C
- added C24, C25: 1u, Capacitor_SMD:C_0402_1005Metric, symbol Device:C
- added C26: 100u, Capacitor_SMD:C_1206_3216Metric, symbol Device:C
- added D4: (no value), symbol Diode:1N4148W
- added D5: LED, LED_SMD:LED_0603_1608Metric, symbol Device:LED
- added IC10: (no value), symbol SamacSys_Parts:NJM2878F3-33-TE2
- added IC9: (no value), symbol SamacSys_Parts:NJM12888F33-TE1
- added R30: (no value), symbol Device:R
- added R31: 1k, Resistor_SMD:R_0402_1005Metric, symbol Device:R
- added U2: (no value), symbol prometheus-schlib:ICM-20948-SL
- C1, C10, C2, C5, C6: LCSC C307331 -> (none)
- C8, C9: LCSC C23630 -> C52923
- D2: LCSC C81598 -> (none)
Connections:
- net +1V8: now also C23.1, IC9.5 (VOUT), U2.1 (VDD), U2.2 (VDDIO), U2.6 (CS)
- net +3V3: now also C22.1, C26.1, IC9.1 (VIN), IC9.3 (CONTROL); no longer IC4.4 (VREF), IC5.4 (VREF)
- net 7V4: now also C24.1, D4.2 (A), IC10.1 (CONTROL), IC10.5 (VIN); no longer C15.1, D2.1 (K), IC8.6 (VIN)
- net GND: now also C22.2, C23.2, C24.2, C25.2, C26.2, D5.1 (K), IC10.2 (GND), IC9.2 (GND), R30.1, U2.10 (GND)
- net GPIO18_MO_B1: now also IC5.2 (IN2); no longer IC5.3 (IN1)
- net GPIO19_MO_B2: now also IC5.3 (IN1); no longer IC5.2 (IN2)
- net GPIO4_GNSS_TX: now also J2.3 (Pin_3); no longer J2.2 (Pin_2)
- net GPIO5_GNSS_RX: now also J2.2 (Pin_2); no longer J2.3 (Pin_3)
- net IMU_SCL: now also U2.3 (SCL)
- net IMU_SDA: now also U2.4 (SDA)
- net RUN: now also IC1.26 (RUN)
- net GPIO8_ToF_SDA: now reaches IC1.11 (GPIO8)
- net GPIO8_ToF_SDA: now also J4.3 (Pin_3)
- net GPIO9_ToF_SCL: now reaches IC1.12 (GPIO9)
- net GPIO9_ToF_SCL: now also J4.2 (Pin_2)
- net GPIO14_IMU_SDA: now reaches IC1.17 (GPIO14)
- net GPIO14_IMU_SDA: now also IC6.D2 (SDA2), R16.2
- net GPIO15_IMU_SCL: now reaches IC1.18 (GPIO15)
- net GPIO15_IMU_SCL: now also IC6.C2 (SCL2), R15.2
- net GPIO17_Nichrome: now reaches IC1.28 (GPIO17)
- net GPIO17_Nichrome: now also R21.1
- net GPIO28_Imonitor: now reaches IC1.40 (GPIO28/ADC2)
- net GPIO28_Imonitor: now also IC7.3 (IN(-)), IC7.4 (OUT)
- net GPIO10_MO_A1: no longer names the net of IC1.13 (GPIO10)
- net GPIO10_MO_A1: no longer IC4.3 (IN1)
- net GPIO11_MO_A2 renamed GPIO14_ToF_RST
- net GPIO14_ToF_RST: now also J4.1 (Pin_1); no longer IC4.2 (IN2)
- removed net GPIO12_IMU_SDA: IC1.15 (GPIO12), IC6.D2 (SDA2), R16.2
- removed net GPIO13_IMU_SCL: IC1.16 (GPIO13), IC6.C2 (SCL2), R15.2
- net GPIO20_MOE_A1 renamed GPIO20_MO_A1
- net GPIO20_MO_A1: now also IC4.2 (IN2); no longer J1.2 (Pin_2)
- net GPIO21_MOE_B1 renamed GPIO21_MO_A2
- net GPIO21_MO_A2: now also IC4.3 (IN1); no longer J3.2 (Pin_2)
- net GPIO22_MOE_A2 renamed GPIO22_MOE_A1
- net GPIO22_MOE_A1: now also J1.2 (Pin_2); no longer J1.3 (Pin_3)
- net GPIO23_MOE_B2 renamed GPIO23_MOE_B1
- net GPIO23_MOE_B1: now also J3.2 (Pin_2); no longer J3.3 (Pin_3)
- net GPIO24_Nichrome renamed GPIO24_MOE_A2
- net GPIO24_MOE_A2: now also J1.3 (Pin_3); no longer R21.1
- net GPIO25_LED renamed GPIO12_LED
- net GPIO12_LED: now also IC1.15 (GPIO12); no longer IC1.37 (GPIO25)
- removed net GPIO26_Imonitor: IC1.38 (GPIO26/ADC0), IC7.3 (IN(-)), IC7.4 (OUT)
- net GPIO3_ToF_RST: no longer names the net of IC1.5 (GPIO3)
- net GPIO3_ToF_RST: no longer J4.2 (Pin_2)
- net GPIO6_ToF_SDA: no longer names the net of IC1.8 (GPIO6)
- net GPIO6_ToF_SDA: no longer J4.3 (Pin_3)
- net GPIO7_ToF_SCL: no longer names the net of IC1.9 (GPIO7)
- net GPIO7_ToF_SCL: no longer J4.1 (Pin_1)
- new net: R30.2, U2.5 (AD0)
- new net: C15.1, D2.1 (K), D4.1 (K), IC8.6 (VIN)
- new net: D5.2 (A), R31.2
- new net 3V3A: C25.1, IC10.4 (VOUT), IC4.4 (VREF), IC5.4 (VREF)
- new net GPIO13_LED: IC1.16 (GPIO13), R31.1
- new net GPIO25_MOE_B2: IC1.37 (GPIO25), J3.3 (Pin_3)
Other:
- moved on the sheet: C14, C15, C16, C17, C18, C19, C20, C21, D2, D3, IC7, IC8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

Commit message: update kicad pcb
Parts:
- removed S1, S2: (no value), symbol SamacSys_Parts:SKRPABE010
- added S1, S2: (no value), symbol SamacSys_Parts:SKRPACE010
- C1, C2: LCSC (none) -> C307331
- C24, C25: value 1u -> (none); footprint Capacitor_SMD:C_0402_1005Metric -> (none)
- C26: value 100u -> (none); footprint Capacitor_SMD:C_1206_3216Metric -> (none)
- D5: value LED -> (none); footprint LED_SMD:LED_0603_1608Metric -> (none)
- R31: value 1k -> (none); footprint Resistor_SMD:R_0402_1005Metric -> (none)
Connections:
- net GND: now also S1.3, S1.4, S2.3, S2.4
- net RUN: now also S2.1, S2.2
- net at R2.1: now also S1.1, S1.2

Commit message: update sch & pcb (em-rev4!)
Parts:
- removed IC6: (no value), symbol SamacSys_Parts:PCA9306YZTR
- removed Q3: (no value), symbol SamacSys_Parts:IRFML8244TRPBF
- removed R23, R26: (no value), symbol Device:R
- added IC6: (no value), symbol SamacSys_Parts:PCA9306DCUR
- added Q3: (no value), symbol SamacSys_Parts:IRLML6402
- R12, R15, R16, R9: LCSC C25879 -> (none)
- R22: LCSC C25744 -> (none)
Connections:
- net GNDA is gone; now on net BAT_IN: J7.1 (Pin_1)
- net +1V8: now also R15.2, R16.2, IC6.2 (VREF1); no longer R12.1, R9.1
- net +3V3: now also R12.1, R9.1; no longer R15.1, R16.1
- net 7V4: now also Q3.3; no longer R27.2
- net BAT_IN: now also R22.1, Q3.2; no longer J7.3 (Pin_3), S3.2
- net GND: now also IC4.9 (EP), IC5.9 (EP), J7.3 (Pin_3), S3.3, IC6.1 (GND)
- net GPIO14_IMU_SDA: now also R12.2, IC6.5 (SDA2); no longer R16.2
- net GPIO15_IMU_SCL: now also R9.2, IC6.6 (SCL2); no longer R15.2
- net GPIO29_Vmonitor: now also Q1.2 (S)
- net IMU_SCL: now also R15.1, IC6.3 (SCL1); no longer R9.2
- net IMU_SDA: now also R16.1, IC6.4 (SDA1); no longer R12.2
- net at C13.1, R8.2: now also IC6.7 (VREF2), IC6.8 (EN)
- net VREG: now reaches C15.1, D2.1 (K), D4.1 (K), IC8.6 (VIN)
- net VREG: now also R27.2
- net at R22.2: now also S3.2, Q3.1
Other:
- note added: "I = Imonitor * 3"
- note added: "VBAT = Vmonitor * 5"
- company: (none) -> DERC CanSat Project
- title: (none) -> Prometheus-EM2a
- moved on the sheet: C16, J7, R30, S3, U2

Commit message: changed level-shifter
Changed lines of the file:
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@@
       (effects (font (size 1.27 1.27)) hide)
     )
-    (property "Value" "" (id 1) (at 275.59 39.37 0))
+    (property "Value" "GND" (id 1) (at 275.59 39.37 0))
     (property "Footprint" "" (id 2) (at 275.59 34.29 0)
       (effects (font (size 1.27 1.27)) hide)
@@
       (effects (font (size 1.27 1.27)) hide)
     )
-    (property "Value" "" (id 1) (at 313.69 30.48 0))
+    (property "Value" "PWR_FLAG" (id 1) (at 313.69 30.48 0))
     (property "Footprint" "" (id 2) (at 313.69 34.29 0)
       (effects (font (size 1.27 1.27)) hide)
@@
       (effects (font (size 1.27 1.27)) hide)
     )
-    (property "Value" "" (id 1) (at 299.72 54.61 0))
+    (property "Value" "GND" (id 1) (at 299.72 54.61 0))
     (property "Footprint" "" (id 2) (at 299.72 50.8 0)
       (effects (font (size 1.27 1.27)) hide)
@@
     )
     (path "/2e989e21-a1e8-42fb-88bc-90b86bc3c254"
-      (reference "Q3") (unit 1) (value "IRLML6402") (footprint "SOT95P237X112-3N")
+      (reference "Q3") (unit 1) (value "IRLML6402") (footprint "SamacSys_Parts:SOT95P237X112-3N")
     )
     (path "/297924c3-c561-498c-9a62-e0aa37bd0634"

Commit message: update main board pcb, add ublox-m10s pcb
Parts:
- added JP1: (no value), symbol Jumper:SolderJumper_2_Open
- added Q4: (no value), symbol SamacSys_Parts:IRLML6402
- added R23: (no value), symbol Device:R
- R10, R11, R13, R14: LCSC (none) -> C22936
Connections:
- net +3V3: now also JP1.1 (A), Q4.2, R23.1; no longer J2.1 (Pin_1)
- net GPIO7_GNSS_RST: now reaches IC1.9 (GPIO7)
- net GPIO7_GNSS_RST: now also Q4.1, R23.2
- new net: J2.1 (Pin_1), JP1.2 (B), Q4.3
Other:
- moved on the sheet: J1, J2, J3, J4, R30, U2

Commit message: add eeprom for log
Parts:
- removed JP1: (no value), symbol Jumper:SolderJumper_2_Open
- added C27: 100n, Capacitor_SMD:C_0603_1608Metric, symbol Device:C
- added IC11: S-24CM01CI-J8T1U4, SOT127P600X175-8N, symbol SamacSys_Parts:S-24CM01CI-J8T1U4
- added Q5: IRLML6402, SamacSys_Parts:SOT95P237X112-3N, symbol SamacSys_Parts:IRLML6402
- added R26: 30k, Resistor_SMD:R_0603_1608Metric, symbol Device:R
- C1, C11, C12, C13, C2, C3, C4, C7: value (none) -> 100n; footprint (none) -> Capacitor_SMD:C_0402_1005Metric
- C10, C5, C6: value (none) -> 100n; footprint (none) -> Capacitor_SMD:C_0603_1608Metric
- C14: value (none) -> 10n; footprint (none) -> Capacitor_SMD:C_0402_1005Metric
- C15, C16: value (none) -> 22u; footprint (none) -> Capacitor_SMD:C_0603_1608Metric
- C17, C18, C19, C20, C21, C26: value (none) -> 100u; footprint (none) -> Capacitor_SMD:C_1206_3216Metric
- C22, C23, C24, C25, C8, C9: value (none) -> 1u; footprint (none) -> Capacitor_SMD:C_0402_1005Metric
- D1, D3, D5: value (none) -> LED; footprint (none) -> LED_SMD:LED_0603_1608Metric
- D2, D4: value (none) -> 1N4148W; footprint (none) -> Diode_SMD:D_SOD-123
- IC1: value (none) -> RP2040; footprint (none) -> SamacSys_Parts:QFN40P700X700X90-57N-D
- IC10: value (none) -> NJM2878F3-33-TE2; footprint (none) -> SamacSys_Parts:SOT65P210X100-5N
- IC2: value (none) -> SIT2001BI-S2-33E-12.000000G; footprint (none) -> SamacSys_Parts:SOT95P280X130-5N
- IC3: value (none) -> W25Q128JVSIQ; footprint (none) -> SamacSys_Parts:SOIC127P790X216-8N
- IC4, IC5: value (none) -> TB67H450FNG,EL; footprint (none) -> SamacSys_Parts:SOIC127P600X175-9N
- IC6: value (none) -> PCA9306DCUR; footprint (none) -> SamacSys_Parts:SOP50P310X90-8N
- IC7: value (none) -> S-89431ACMC-HBVT2U; footprint (none) -> SamacSys_Parts:SOT95P275X130-5N
- IC8: value (none) -> NJM2884U1-33-TE1; footprint (none) -> SamacSys_Parts:SOT-89-5-1
- IC9: value (none) -> NJM12888F33-TE1; footprint (none) -> SamacSys_Parts:SOT95P280X130-5N
- J1: value (none) -> MOE_A; footprint (none) -> tanekonsat:PinHeader_1x04_P2.00mm_Vertical
- J2: value (none) -> GNSS; footprint (none) -> Connector_JST_ZH:JST_ZH_B4B-ZR_1x04_P1.50mm_Vertical
- J3: value (none) -> MOE_B; footprint (none) -> tanekonsat:PinHeader_1x04_P2.00mm_Vertical
- J4: value (none) -> ToF; footprint (none) -> Connector_JST_ZH:JST_ZH_B5B-ZR_1x05_P1.50mm_Vertical
- J5: value (none) -> Motor1; footprint (none) -> Connector_PinHeader_2.00mm:PinHeader_1x02_P2.00mm_Vertical
- J6: value (none) -> Motor2; footprint (none) -> Connector_PinHeader_2.00mm:PinHeader_1x02_P2.00mm_Vertical
- J7: value (none) -> JST_PH_3_Side; footprint (none) -> Connectors_JST:JST_PH_S3B-PH-K_03x2.00mm_Angled
- J8: value (none) -> Nichrome; footprint (none) -> Connector_PinHeader_2.00mm:PinHeader_1x02_P2.00mm_Vertical
- Q1, Q2: value (none) -> IRFML8244TRPBF; footprint (none) -> SamacSys_Parts:SOT95P237X112-3N
- Q3, Q4: value (none) -> IRLML6402; footprint (none) -> SamacSys_Parts:SOT95P237X112-3N
- R1, R2, R21, R28, R31, R7: value (none) -> 1k; footprint (none) -> Resistor_SMD:R_0402_1005Metric
- R10, R11, R13, R14: value (none) -> 1; footprint (none) -> Resistor_SMD:R_0603_1608Metric
- R12, R15, R16, R9: value (none) -> 2.2k; footprint (none) -> Resistor_SMD:R_0402_1005Metric
- R17, R23: value (none) -> 30k; footprint (none) -> Resistor_SMD:R_0603_1608Metric
- R18, R24, R27, R30: value (none) -> 10k; footprint (none) -> Resistor_SMD:R_0402_1005Metric
- R19, R20: value (none) -> 100; footprint (none) -> Resistor_SMD:R_0402_1005Metric
- R22: value (none) -> 100k; footprint (none) -> Resistor_SMD:R_0402_1005Metric
- R25: value (none) -> 3k; footprint (none) -> Resistor_SMD:R_0603_1608Metric
- R29: value (none) -> 0.01; footprint (none) -> Resistor_SMD:R_1206_3216Metric
- R3: value (none) -> 5.1k; footprint (none) -> Resistor_SMD:R_0402_1005Metric
- R5, R6: value (none) -> 27; footprint (none) -> Resistor_SMD:R_0402_1005Metric
- R8: value (none) -> 200k; footprint (none) -> Resistor_SMD:R_0402_1005Metric
- S1, S2: value (none) -> SKRPACE010; footprint (none) -> SamacSys_Parts:SMT_4.2X3.2_
- S3: value (none) -> SSSS811101; footprint (none) -> SamacSys_Parts:SSSS811101
- U1: value (none) -> USB_type_C; footprint (none) -> tanekonsat:USB_typeC_t
- U2: value (none) -> ICM-20948-SL; footprint (none) -> tanekonsat:ICM-20948_SL
- U3: value (none) -> LT6106; footprint (none) -> Package_TO_SOT_SMD:SOT-23-5
Connections:
- net +1V8: now also C27.1, IC11.8 (VCC)
- net +3V3: now also Q5.2, R26.1; no longer J4.4 (Pin_4)
- net GND: now also C27.2, IC11.1 (NC), IC11.2 (A1), IC11.3 (A2), IC11.4 (GND), IC11.7 (WP)
- net IMU_SCL: now also IC11.6 (SCL)
- net IMU_SDA: now also IC11.5 (SDA)
- net GPIO10_ToF_LPn: now reaches IC1.13 (GPIO10)
- net GPIO10_ToF_LPn: now also J4.1 (Pin_1)
- net GPIO14_ToF_RST renamed GPIO14_ToF_VCC
- net GPIO14_ToF_VCC: now also Q5.1, R26.2; no longer J4.1 (Pin_1)
- net GPIO7_GNSS_RST renamed GPIO7_GNSS_VCC
- new net: J4.4 (Pin_4), Q5.3
Other:
- note added: "Memory"
- moved on the sheet: IC4, IC5, J1, J3, J5, J6, R10, R11, R13, R14
