File: kicad2/prometheus-em/prometheus-em.kicad_sch (KiCad schematic)
At the start: 93 parts, among them IC1 RP2040, IC10 NJM2878F3-33-TE2, IC11 S-24CM01CI-J8T1U4, IC2 SIT2001BI-S2-33E-12.000000G, IC3 W25Q128JVSIQ, IC4 TB67H450FNG,EL, IC5 TB67H450FNG,EL, IC6 PCA9306DCUR, IC7 S-89431ACMC-HBVT2U, IC8 NJM2884U1-33-TE1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

Commit message: add ir feature
Parts:
- removed C26: 100u, Capacitor_SMD:C_1206_3216Metric, symbol Device:C
- removed D5: LED, LED_SMD:LED_0603_1608Metric, symbol Device:LED
- removed R31: 1k, Resistor_SMD:R_0402_1005Metric, symbol Device:R
- added J10: (no value), symbol Connector:Conn_01x03_Male
- added J9: (no value), symbol Connector:Conn_01x02_Male
- added Q6: IRLML6402, SamacSys_Parts:SOT95P237X112-3N, symbol SamacSys_Parts:IRLML6402
- added R32: 30k, Resistor_SMD:R_0603_1608Metric, symbol Device:R
- added R33: (no value), symbol Device:R
- C1: value 100n -> (none); footprint Capacitor_SMD:C_0402_1005Metric -> (none)
- R4: value (none) -> 5.1k; footprint (none) -> Resistor_SMD:R_0402_1005Metric
Connections:
- net +3V3: now also J10.1 (Pin_1), Q6.2, R32.1
- net 7V4: no longer Q3.3
- net BAT_IN: now also Q3.3; no longer J7.1 (Pin_1), Q3.2, R22.1
- net GND: now also J10.2 (Pin_2), J9.1 (Pin_1)
- net GPIO2_LED: now reaches IC1.4 (GPIO2)
- net GPIO2_LED: now also R7.1
- net GPIO3_LED: now reaches IC1.5 (GPIO3)
- net GPIO12_LED renamed GPIO12_IR_IN
- net GPIO12_IR_IN: now also J10.3 (Pin_3); no longer R7.1
- net GPIO13_LED renamed GPIO12_IR_OUT
- net GPIO12_IR_OUT: now also Q6.1, R32.2
- new net: Q6.3, R33.1
- new net: J9.2 (Pin_2), R33.2
- new net: J7.1 (Pin_1), Q3.2, R22.1
Other:
- note added: "IR"
- moved on the sheet: C18
